File: cad_files/mm7d/mm7d.kicad_pcb (KiCad board)
At the start: 2 copper layers, 52.8 x 63.5 mm, 26 parts, among them P101 CONN_01X02, P102 CONN_01X02, U101-JP4 CONN_01X10, U101-JP5 CONN_01X10, U102 MQ-135M, U103 DHT11

Commit message: 230317
Parts:
- removed REF** (x4): MountingHole_2.5mm, mm7d:MyMountingHole_2.5mm
- removed U103: DHT11, Socket_Strips:Socket_Strip_Straight_1x04
- R107: value 39k -> 5.1k
- R108: value 9.1k -> 750
- U102: value MQ-135M -> DHT11
- moved U102 54.3 mm to (146.1, 127.0), turned to 0 degrees
Connections:
- R107 pad 1: Net-(R107-Pad1) -> +5V
- U102 pad 1: +5V -> +3V3
- U102 pad 2: GND -> Net-(R106-Pad2)
- U102 pad 4: Net-(R107-Pad1) -> GND
Routing:
- net Net-(R107-Pad1): track 19.6 -> 0.00 mm
- net +5V: track 101.8 -> 82.6 mm, vias 1 -> 0
- net GND: track 154.0 -> 135.7 mm
Other:
- board text added: "2023"
- board text removed: "2020"
- board text removed: "Dn.: 59/12/3"
