File: cad_files/mm7d/mm7d.sch (KiCad schematic (older format))
At the start: 23 parts, among them K1 electromagnetic_actor_1, K1a switch_alt_1P, P1 BNC, P2 DB9, Q1 BD139, U1 Adafruit Huzzah Breakout, U2 MQ-135M, U3 DHT11

Commit message: 200620
Parts:
- removed Q1: BD139, symbol Q_NPN_ECB
- added Q1: 2N4401, symbol Q_NPN_EBC
- K1: value electromagnetic_actor_1 -> RSY-5
- R5: value 4k -> 100k
- R6: value 1k -> 24k
Connections:
- wire segments 72 -> 57
- no-connect marks 22 -> 24
Changed lines of the file:
@@
 U 1 1 5EEE159B
 P 6000 4700
-F 0 "U1" H 5550 5450 60  0000 C CNN
-F 1 "Adafruit Huzzah Breakout" H 6000 3950 60  0000 C CNN
+F 0 "U1" H 5550 5450 50  0000 C CNN
+F 1 "Adafruit Huzzah Breakout" H 6000 3950 50  0000 C CNN
 F 2 "" H 5850 4470 60  0001 C CNN
 F 3 "" H 5850 4470 60  0001 C CNN
@@
 $EndComp
 Wire Wire Line
-	4400 2000 4400 2050
-Wire Wire Line
-	4400 2050 4400 2200
-Wire Wire Line
-	4600 1800 4600 2050
-Wire Wire Line
-	4600 2050 4600 2200
+	4400 2000 4400 2200
+Wire Wire Line
+	4600 1800 4600 2200
 Wire Wire Line
 	4600 1800 4550 1800
 $Comp
-L 0V #PWR13
+L 0V #PWR01
 U 1 1 5EEE1D86
 P 8150 5450
-F 0 "#PWR13" H 8150 5200 50  0001 C CNN
+F 0 "#PWR01" H 8150 5200 50  0001 C CNN
 F 1 "0V" H 8150 5300 50  0001 C CNN
 F 2 "" H 8150 5450 50  0000 C CNN
@@
 $EndComp
 Wire Wire Line
-	8150 3750 8150 4850
-Wire Wire Line
-	8150 4850 8150 5450
+	8150 3750 8150 5450
 $Comp
 L fuse F1
@@
 $EndComp
 Wire Wire Line
-	4600 3050 4600 3200
-Wire Wire Line
-	4600 3200 4600 3650
-Wire Wire Line
-	4600 3650 4600 4300
-Wire Wire Line
-	5950 3500 5950 3650
-Wire Wire Line
-	5950 3650 5950 3800
-Wire Wire Line
-	4600 3650 5950 3650
-Wire Wire Line
-	5950 3650 8300 3650
+	4600 3050 4600 4300
+Wire Wire Line
+	5950 3500 5950 3800
+Wire Wire Line
+	4600 3650 8300 3650
 Connection ~ 4600 3200
 NoConn ~ 5850 3800
@@
 	5750 2400 5750 3800
 $Comp
-L 0V #PWR6
+L 0V #PWR02
 U 1 1 5EEE2266
 P 4150 3200
-F 0 "#PWR6" H 4150 2950 50  0001 C CNN
+F 0 "#PWR02" H 4150 2950 50  0001 C CNN
 F 1 "0V" H 4150 3050 50  0001 C CNN
 F 2 "" H 4150 3200 50  0000 C CNN
@@
 	4200 3200 4150 3200
 $Comp
-L 0V #PWR5
+L 0V #PWR03
 U 1 1 5EEE22DD
 P 4150 2750
-F 0 "#PWR5" H 4150 2500 50  0001 C CNN
+F 0 "#PWR03" H 4150 2500 50  0001 C CNN
 F 1 "0V" H 4150 2600 50  0001 C CNN
 F 2 "" H 4150 2750 50  0000 C CNN
@@
 Connection ~ 4600 2050
 $Comp
-L +5V #PWR11
+L +5V #PWR04
 U 1 1 5EEE284E
 P 5950 3500
-F 0 "#PWR11" H 5950 3350 50  0001 C CNN
+F 0 "#PWR04" H 5950 3350 50  0001 C CNN
 F 1 "+5V" H 5950 3650 50  0000 C CNN
 F 2 "" H 5950 3500 50  0000 C CNN
@@
 	5450 2400 5750 2400
 $Comp
-L 0V #PWR12
+L 0V #PWR05
 U 1 1 5EEE2C07
 P 6800 4250
-F 0 "#PWR12" H 6800 4000 50  0001 C CNN
+F 0 "#PWR05" H 6800 4000 50  0001 C CNN
 F 1 "0V" H 6800 4100 50  0001 C CNN
 F 2 "" H 6800 4250 50  0000 C CNN
@@
 NoConn ~ 6700 4950
 $Comp
-L +3.3V #PWR10
+L +3.3V #PWR06
 U 1 1 5EEE2DDF
 P 5100 3500
-F 0 "#PWR10" H 5100 3350 50  0001 C CNN
+F 0 "#PWR06" H 5100 3350 50  0001 C CNN
 F 1 "+3.3V" H 5100 3650 50  0000 C CNN
 F 2 "" H 5100 3500 50  0000 C CNN
@@
 $EndComp
 $Comp
-L Q_NPN_ECB Q1
-U 1 1 5EEE3306
-P 3850 4750
-F 0 "Q1" H 3750 4550 50  0000 L CNN
-F 1 "BD139" H 3600 4950 50  0000 L CNN
-F 2 "" H 4050 4850 50  0000 C CNN
-F 3 "" H 3850 4750 50  0000 C CNN
-	1    3850 4750
-	-1   0    0    -1
-$EndComp
-$Comp
 L electromagnetic_actor_1 K1
 U 1 1 5EEE3451
 P 3750 4150
-F 0 "K1" H 4000 4350 50  0000 L CNN
-F 1 "electromagnetic_actor_1" H 3800 4100 50  0001 L CNN
+F 0 "K1" H 3950 4300 50  0000 L CNN
+F 1 "RSY-5" H 3900 4100 50  0000 L CNN
 F 2 "" V 3725 4250 50  0001 C CNN
 F 3 "" V 3725 4250 50  0001 C CNN
@@
 $EndComp
 Wire Wire Line
-	6700 4650 7800 4650
-Wire Wire Line
-	7800 4650 8300 4650
+	6700 4650 8300 4650
 Wire Wire Line
 	7800 4550 7800 4650
@@
 	7800 4250 7800 4150
 Wire Wire Line
-	3750 4250 3750 4300
-Wire Wire Line
-	3750 4300 3750 4550
+	3750 4250 3750 4550
 Wire Wire Line
 	3750 4300 4000 4300
@@
 Connection ~ 3750 4300
 Wire Wire Line
-	3750 3500 3750 3900
-Wire Wire Line
-	3750 3900 3750 3950
+	3750 3500 3750 3950
 Wire Wire Line
 	3750 3900 4000 3900
@@
 	5300 4750 4400 4750
 $Comp
-L +5V #PWR3
+L +5V #PWR07
 U 1 1 5EEE3F2D
 P 3750 3500
-F 0 "#PWR3" H 3750 3350 50  0001 C CNN
+F 0 "#PWR07" H 3750 3350 50  0001 C CNN
 F 1 "+5V" H 3750 3650 50  0000 C CNN
 F 2 "" H 3750 3500 50  0000 C CNN
@@
 Connection ~ 3750 3900
 $Comp
-L 0V #PWR4
+L 0V #PWR08
 U 1 1 5EEE4100
 P 3750 5450
-F 0 "#PWR4" H 3750 5200 50  0001 C CNN
+F 0 "#PWR08" H 3750 5200 50  0001 C CNN
 F 1 "0V" H 3750 5300 50  0001 C CNN
 F 2 "" H 3750 5450 50  0000 C CNN
@@
 	4850 4650 4900 4650
 $Comp
-L 0V #PWR9
+L 0V #PWR09
 U 1 1 5EEE442D
 P 4850 5450
-F 0 "#PWR9" H 4850 5200 50  0001 C CNN
+F 0 "#PWR09" H 4850 5200 50  0001 C CNN
 F 1 "0V" H 4850 5300 50  0001 C CNN
 F 2 "" H 4850 5450 50  0000 C CNN
@@
 $EndComp
 $Comp
-L 0V #PWR8
+L 0V #PWR010
 U 1 1 5EEE45B4
 P 4600 5450
-F 0 "#PWR8" H 4600 5200 50  0001 C CNN
+F 0 "#PWR010" H 4600 5200 50  0001 C CNN
 F 1 "0V" H 4600 5300 50  0001 C CNN
 F 2 "" H 4600 5450 50  0000 C CNN
@@
 $EndComp
 $Comp
-L 0V #PWR2
+L 0V #PWR011
 U 1 1 5EEE4B4D
 P 3300 5450
-F 0 "#PWR2" H 3300 5200 50  0001 C CNN
+F 0 "#PWR011" H 3300 5200 50  0001 C CNN
 F 1 "0V" H 3300 5300 50  0001 C CNN
 F 2 "" H 3300 5450 50  0000 C CNN
@@
 	3300 4600 3300 4550
 $Comp
-L +3.3V #PWR1
+L +3.3V #PWR012
 U 1 1 5EEE5097
 P 3200 3500
-F 0 "#PWR1" H 3200 3350 50  0001 C CNN
+F 0 "#PWR012" H 3200 3350 50  0001 C CNN
 F 1 "+3.3V" H 3200 3650 50  0000 C CNN
 F 2 "" H 3200 3500 50  0000 C CNN
@@
 	8050 4550 8050 4150
 Wire Wire Line
-	8050 4150 7800 4150
-Wire Wire Line
-	7800 4150 7500 4150
+	8050 4150 7500 4150
 Wire Wire Line
 	3100 5650 7500 5650
@@
 P 7050 5250
 F 0 "R6" H 7150 5300 50  0000 L CNN
-F 1 "1k" H 7150 5200 50  0000 L CNN
+F 1 "24k" H 7150 5200 50  0000 L CNN
 F 2 "" V 6980 5250 50  0000 C CNN
 F 3 "" H 7050 5250 50  0000 C CNN
@@
 $EndComp
 Wire Wire Line
-	7050 5000 7050 5050
-Wire Wire Line
-	7050 5050 7050 5100
+	7050 5000 7050 5100
 Wire Wire Line
 	6700 5050 7050 5050
 Connection ~ 7050 5050
 $Comp
-L 0V #PWR?
+L 0V #PWR013
 U 1 1 5EEEB31B
 P 7050 5450
-F 0 "#PWR?" H 7050 5200 50  0001 C CNN
+F 0 "#PWR013" H 7050 5200 50  0001 C CNN
 F 1 "0V" H 7050 5300 50  0001 C CNN
 F 2 "" H 7050 5450 50  0000 C CNN
@@
 	7050 5400 7050 5450
 Wire Wire Line
-	6700 4750 6950 4750
-Wire Wire Line
-	6950 4750 6950 3850
-Wire Wire Line
-	6950 3850 8300 3850
-Wire Wire Line
 	8300 3950 7050 3950
 Wire Wire Line
@@
 P 7050 4850
 F 0 "R5" H 7150 4900 50  0000 L CNN
-F 1 "4k" H 7150 4800 50  0000 L CNN
+F 1 "100k" H 7150 4800 50  0000 L CNN
 F 2 "" V 6980 4850 50  0000 C CNN
 F 3 "" H 7050 4850 50  0000 C CNN
@@
 	1    0    0    -1
 $EndComp
+NoConn ~ 8300 3850
+NoConn ~ 6700 4750
+$Comp
+L Q_NPN_EBC Q1
+U 1 1 5EEE5F0C
+P 3850 4750
+F 0 "Q1" H 3700 4900 50  0000 L CNN
+F 1 "2N4401" H 3600 4500 50  0000 L CNN
+F 2 "" H 4050 4850 50  0000 C CNN
+F 3 "" H 3850 4750 50  0000 C CNN
+	1    3850 4750
+	-1   0    0    -1
+$EndComp
 $EndSCHEMATC

Commit message: 200621
Parts:
- R5: value 100k -> 39k
- R6: value 24k -> 9.1k
Changed lines of the file:
@@
 P 7050 5250
 F 0 "R6" H 7150 5300 50  0000 L CNN
-F 1 "24k" H 7150 5200 50  0000 L CNN
+F 1 "9.1k" H 7150 5200 50  0000 L CNN
 F 2 "" V 6980 5250 50  0000 C CNN
 F 3 "" H 7050 5250 50  0000 C CNN
@@
 P 7050 4850
 F 0 "R5" H 7150 4900 50  0000 L CNN
-F 1 "100k" H 7150 4800 50  0000 L CNN
+F 1 "39k" H 7150 4800 50  0000 L CNN
 F 2 "" V 6980 4850 50  0000 C CNN
 F 3 "" H 7050 4850 50  0000 C CNN

Commit message: 200627
Parts:
- removed D2: LED, symbol LED
- removed K1a: switch_alt_1P, symbol switch_alt_1P
- removed R1: 360, symbol R
- added C2: 1000u, symbol CP_Small
- added D5: green, symbol LED
- added D6: yellow, symbol LED
- added D7: red, symbol LED
- added R2, R5, R6: 360, symbol R
- added SW1: switch_1P_closed, symbol switch_1P_closed
- D3: value LED -> white
- D4: value LED -> blue
- renumbered D5 to D2, R3 to R1, R4 to R3, R2 to R4, R5 to R7, R6 to R8, R7 to R9
Connections:
- wire segments 57 -> 66
- no-connect marks 24 -> 21
Other:
- note added: "5V DC in"
- note added: "Console (3,3V serial)"
- note added: "PCB"
- note added: "Power Act Status"
- note added: "ferrite ring"
- note removed: ""5V DC IN""
- note removed: ""ACT""
- note removed: ""CONSOLE""
- note removed: ""POWER""
- note removed: ""SENSOR\n ERROR""
- moved on the sheet: C1, D1, D2, D3, F1, K1, L1, P1, P2, Q1, R1, R3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

Commit message: 200628
Parts:
- removed D3: white, symbol LED
- removed D4: blue, symbol LED
- removed D5: green, symbol LED
- removed D6: yellow, symbol LED
- removed D7: red, symbol LED
- added D3: white, symbol LED-CIRCLE
- added D4: blue, symbol LED-CIRCLE
- added D5: green, symbol LED-CIRCLE
- added D6: yellow, symbol LED-CIRCLE
- added D7: red, symbol LED-CIRCLE
- R1: value 470 -> 680
- R2, R3, R5, R6: value 360 -> 470
Connections:
- wire segments 66 -> 82
Other:
- moved on the sheet: D2, R3, R4, R5, R6

Commit message: 200629
Parts:
- added C3: 2.2u, symbol CP_Small
- added Sp1: Speaker Crystal, symbol Speaker_Ultrasound
Connections:
- net GND: now also Sp1.2
- net at U1.4/5 (#14): now also C3.1
- new net: C3.2, Sp1.1
- no-connect marks 21 -> 20
Other:
- moved on the sheet: R7, R8, R9, U2, U3
Changed lines of the file:
@@
 L DHT11 U3
 U 1 1 5EEE15C4
-P 9125 4700
-F 0 "U3" H 9025 4950 50  0000 C CNN
-F 1 "DHT11" H 9125 4450 50  0000 C CNN
-F 2 "" H 9275 4950 50  0001 C CNN
-F 3 "" H 9275 4950 50  0001 C CNN
-	1    9125 4700
+P 9225 4700
+F 0 "U3" H 9125 4950 50  0000 C CNN
+F 1 "DHT11" H 9225 4450 50  0000 C CNN
+F 2 "" H 9375 4950 50  0001 C CNN
+F 3 "" H 9375 4950 50  0001 C CNN
+	1    9225 4700
 	1    0    0    -1
 $EndComp
@@
 L 0V #PWR01
 U 1 1 5EEE1D86
-P 8725 5500
-F 0 "#PWR01" H 8725 5250 50  0001 C CNN
-F 1 "0V" H 8725 5350 50  0001 C CNN
-F 2 "" H 8725 5500 50  0000 C CNN
-F 3 "" H 8725 5500 50  0000 C CNN
-	1    8725 5500
+P 8825 5500
+F 0 "#PWR01" H 8825 5250 50  0001 C CNN
+F 1 "0V" H 8825 5350 50  0001 C CNN
+F 2 "" H 8825 5500 50  0000 C CNN
+F 3 "" H 8825 5500 50  0000 C CNN
+	1    8825 5500
 	1    0    0    -1
 $EndComp
@@
 L +5V #PWR04
 U 1 1 5EEE284E
-P 7725 3200
-F 0 "#PWR04" H 7725 3050 50  0001 C CNN
-F 1 "+5V" H 7725 3350 50  0000 C CNN
-F 2 "" H 7725 3200 50  0000 C CNN
-F 3 "" H 7725 3200 50  0000 C CNN
-	1    7725 3200
+P 7825 3200
+F 0 "#PWR04" H 7825 3050 50  0001 C CNN
+F 1 "+5V" H 7825 3350 50  0000 C CNN
+F 2 "" H 7825 3200 50  0000 C CNN
+F 3 "" H 7825 3200 50  0000 C CNN
+	1    7825 3200
 	1    0    0    -1
 $EndComp
@@
 L R R9
 U 1 1 5EEE8D51
-P 7900 5125
-F 0 "R9" H 7975 5175 50  0000 L CNN
-F 1 "4.7k" H 7975 5075 50  0000 L CNN
-F 2 "" V 7830 5125 50  0000 C CNN
-F 3 "" H 7900 5125 50  0000 C CNN
-	1    7900 5125
+P 8000 5125
+F 0 "R9" H 8075 5175 50  0000 L CNN
+F 1 "4.7k" H 8075 5075 50  0000 L CNN
+F 2 "" V 7930 5125 50  0000 C CNN
+F 3 "" H 8000 5125 50  0000 C CNN
+	1    8000 5125
 	1    0    0    -1
 $EndComp
@@
 Text Notes 5975 1500 0    60   ~ 0
 Console (3,3V serial)
-NoConn ~ 8875 4750
+NoConn ~ 8975 4750
 $Comp
 L MQ-135M U2
 U 1 1 5EEEA952
-P 9125 3800
-F 0 "U2" H 9025 4050 50  0000 C CNN
-F 1 "MQ-135M" H 9125 3550 50  0000 C CNN
-F 2 "" H 8995 4020 50  0001 C CNN
-F 3 "" H 8995 4020 50  0001 C CNN
-	1    9125 3800
+P 9225 3800
+F 0 "U2" H 9125 4050 50  0000 C CNN
+F 1 "MQ-135M" H 9225 3550 50  0000 C CNN
+F 2 "" H 9095 4020 50  0001 C CNN
+F 3 "" H 9095 4020 50  0001 C CNN
+	1    9225 3800
 	1    0    0    -1
 $EndComp
@@
 L R R8
 U 1 1 5EEEB0AE
-P 7625 5250
-F 0 "R8" H 7700 5300 50  0000 L CNN
-F 1 "9.1k" H 7700 5200 50  0000 L CNN
-F 2 "" V 7555 5250 50  0000 C CNN
-F 3 "" H 7625 5250 50  0000 C CNN
-	1    7625 5250
+P 7725 5250
+F 0 "R8" H 7800 5300 50  0000 L CNN
+F 1 "9.1k" H 7800 5200 50  0000 L CNN
+F 2 "" V 7655 5250 50  0000 C CNN
+F 3 "" H 7725 5250 50  0000 C CNN
+	1    7725 5250
 	1    0    0    -1
 $EndComp
@@
 L 0V #PWR012
 U 1 1 5EEEB31B
-P 7625 5500
-F 0 "#PWR012" H 7625 5250 50  0001 C CNN
-F 1 "0V" H 7625 5350 50  0001 C CNN
-F 2 "" H 7625 5500 50  0000 C CNN
-F 3 "" H 7625 5500 50  0000 C CNN
-	1    7625 5500
+P 7725 5500
+F 0 "#PWR012" H 7725 5250 50  0001 C CNN
+F 1 "0V" H 7725 5350 50  0001 C CNN
+F 2 "" H 7725 5500 50  0000 C CNN
+F 3 "" H 7725 5500 50  0000 C CNN
+	1    7725 5500
 	1    0    0    -1
 $EndComp
@@
 L R R7
 U 1 1 5EEEB91E
-P 7625 4850
-F 0 "R7" H 7700 4900 50  0000 L CNN
-F 1 "39k" H 7700 4800 50  0000 L CNN
-F 2 "" V 7555 4850 50  0000 C CNN
-F 3 "" H 7625 4850 50  0000 C CNN
-	1    7625 4850
-	1    0    0    -1
-$EndComp
-NoConn ~ 8875 3850
-NoConn ~ 7325 4750
+P 7725 4850
+F 0 "R7" H 7800 4900 50  0000 L CNN
+F 1 "39k" H 7800 4800 50  0000 L CNN
+F 2 "" V 7655 4850 50  0000 C CNN
+F 3 "" H 7725 4850 50  0000 C CNN
+	1    7725 4850
+	1    0    0    -1
+$EndComp
+NoConn ~ 8975 3850
 $Comp
 L Q_NPN_EBC Q1
@@
 	3675 1800 3625 1800
 Wire Wire Line
-	8725 3750 8725 4850
-Wire Wire Line
-	8725 4850 8725 5500
+	8825 3750 8825 4850
+Wire Wire Line
+	8825 4850 8825 5500
 Wire Wire Line
 	3675 2600 3675 2950
@@
 	5825 4450 5675 4450
 Wire Wire Line
-	7900 5650 7900 5275
-Wire Wire Line
-	7900 4975 7900 4650
+	8000 5650 8000 5275
+Wire Wire Line
+	8000 4975 8000 4650
 Wire Wire Line
 	2975 4250 2975 4300
@@
 	5675 4450 5675 3200
 Wire Wire Line
-	8175 4550 8875 4550
-Wire Wire Line
-	2425 5650 7900 5650
-Wire Wire Line
-	7900 5650 8175 5650
-Connection ~ 7900 4650
-Wire Wire Line
-	8725 4850 8875 4850
-Wire Wire Line
-	8725 3750 8875 3750
-Connection ~ 8725 4850
-Wire Wire Line
-	7625 5000 7625 5050
-Wire Wire Line
-	7625 5050 7625 5100
-Wire Wire Line
-	7325 5050 7625 5050
-Connection ~ 7625 5050
-Wire Wire Line
-	7625 5400 7625 5500
-Wire Wire Line
-	8875 3950 7625 3950
-Wire Wire Line
-	7625 3950 7625 4700
+	8275 4550 8975 4550
+Wire Wire Line
+	2425 5650 8000 5650
+Wire Wire Line
+	8000 5650 8275 5650
+Connection ~ 8000 4650
+Wire Wire Line
+	8825 4850 8975 4850
+Wire Wire Line
+	8825 3750 8975 3750
+Connection ~ 8825 4850
+Wire Wire Line
+	7725 5000 7725 5050
+Wire Wire Line
+	7725 5050 7725 5100
+Wire Wire Line
+	7325 5050 7725 5050
+Connection ~ 7725 5050
+Wire Wire Line
+	7725 5400 7725 5500
+Wire Wire Line
+	8975 3950 7725 3950
+Wire Wire Line
+	7725 3950 7725 4700
 Text Notes 9350 2850 0    60   ~ 0
 PCB
@@
 ferrite ring
 Wire Wire Line
-	7325 4650 7900 4650
-Wire Wire Line
-	7900 4650 8875 4650
-Wire Wire Line
-	8175 5650 8175 4550
-Connection ~ 7900 5650
-Wire Wire Line
-	7725 3200 7725 3650
-Wire Wire Line
-	7725 3650 7725 4450
-Wire Wire Line
-	7725 4450 7325 4450
-Wire Wire Line
-	8875 3650 7725 3650
-Connection ~ 7725 3650
+	7325 4650 8000 4650
+Wire Wire Line
+	8000 4650 8975 4650
+Wire Wire Line
+	8275 5650 8275 4550
+Connection ~ 8000 5650
+Wire Wire Line
+	7825 3200 7825 3650
+Wire Wire Line
+	7825 3650 7825 4450
+Wire Wire Line
+	7825 4450 7325 4450
+Wire Wire Line
+	8975 3650 7825 3650
+Connection ~ 7825 3650
 NoConn ~ 6525 3750
 Connection ~ 5935 1880
@@
 	0    -1   -1   0
 $EndComp
+Wire Wire Line
+	7325 4750 7625 4750
+Wire Wire Line
+	7625 4750 7625 3500
+Wire Wire Line
+	7625 3500 5275 3500
+Wire Wire Line
+	5275 2400 5275 3050
+$Comp
+L CP_Small C3
+U 1 1 5EFA265C
+P 5275 3150
+F 0 "C3" H 5400 3075 50  0000 L CNN
+F 1 "2.2u" H 5400 3200 50  0000 L CNN
+F 2 "" H 5275 3150 50  0000 C CNN
+F 3 "" H 5275 3150 50  0000 C CNN
+	1    5275 3150
+	-1   0    0    1
+$EndComp
+$Comp
+L 0V #PWR?
+U 1 1 5EFA2B1B
+P 5175 2850
+F 0 "#PWR?" H 5175 2600 50  0001 C CNN
+F 1 "0V" H 5175 2700 50  0001 C CNN
+F 2 "" H 5175 2850 50  0000 C CNN
+F 3 "" H 5175 2850 50  0000 C CNN
+	1    5175 2850
+	1    0    0    -1
+$EndComp
+Wire Wire Line
+	5175 2400 5175 2850
+$Comp
+L Speaker_Ultrasound Sp1
+U 1 1 5EFA2C83
+P 5275 2200
+F 0 "Sp1" V 5525 2225 50  0000 R CNN
+F 1 "Speaker Crystal" H 5300 2350 50  0001 R CNN
+F 2 "" H 5240 2150 50  0000 C CNN
+F 3 "" H 5240 2150 50  0000 C CNN
+	1    5275 2200
+	0    1    -1   0
+$EndComp
+Wire Wire Line
+	5275 3500 5275 3250
 $EndSCHEMATC
