File: cad_files/mm7d/mm7d.sch (KiCad schematic (older format))
At the start: 30 parts, among them K1 RSY-5, P1 BNC, P2 DB9, Q1 2N4401, SW1 switch_1P_closed, U1 Adafruit Huzzah Breakout, U2 MQ-135M, U3 DHT11

Commit message: 200705
Parts:
- removed D2: 1N4001, symbol diode
- removed F1: 500mA F, symbol fuse
- removed K1: RSY-5, symbol electromagnetic_actor_1
- removed Q1: 2N4401, symbol Q_NPN_EBC
- removed R4: 1k, symbol R
- removed SW1: switch_1P_closed, symbol switch_1P_closed
- C1: symbol C_Small -> device:C_Small
- C2, C3: symbol CP_Small -> device:CP_Small
- D1: symbol diode -> pzs_others:diode
- D3, D4, D5, D6, D7: symbol LED-CIRCLE -> pzs_devices:LED-CIRCLE
- L1: symbol EMI_Filter_LL -> device:EMI_Filter_LL
- P1: symbol BNC -> mm7d-rescue:BNC
- P2: symbol DB9 -> mm7d-rescue:DB9
- R1, R2, R3, R7, R8: symbol R -> device:R
- R4: renamed from R5; symbol R -> device:R
- R5: renamed from R6; symbol R -> device:R
- R6: renamed from R9; symbol R -> device:R
- Sp1: symbol Speaker_Ultrasound -> device:Speaker_Ultrasound
- U1: symbol Adafruit_Huzzah_Breakout -> pzs_devices:Adafruit_Huzzah_Breakout
- U2: symbol MQ-135M -> pzs_devices:MQ-135M
- U3: symbol DHT11 -> pzs_devices:DHT11
Connections:
- net +3V3: now also R6.1, U3.1 (VCC)
- net +5V: now also C2.1, L1.2
- net at U1.4/6 (#12), U3.2 (IO): now also R6.2; no longer R6.1
- net at U1.4/7 (#13): no longer R2.1
- net at U1.5/5 (#2): now also R2.1; no longer R3.2
- net at U1.5/6 (#0): now also R3.2
- net at R3.1: now also D5.2 (A); no longer D4.2 (A)
- net at R4.1: now also D6.2 (A); no longer D5.2 (A)
- net at R5.1: now also D7.2 (A); no longer D6.2 (A)
- net at R2.2: now also D4.2 (A); no longer D7.2 (A)
- no-connect marks 20 -> 21
Other:
- moved on the sheet: C1, C2, C3, D1, D3, D4, D5, D6, D7, L1, P1, P2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

Commit message: 200705
Parts:
- R1: value 680 -> 470
- renumbered D3 to D2, D4 to D3, D5 to D4, D6 to D5, D7 to D6
Connections:
- net +3V3: now also R1.1
- net +5V: no longer R1.1
Other:
- moved on the sheet: R2, R3, R4, R5
Changed lines of the file:
@@
 L power:+3.3V #PWR06
 U 1 1 5EEE2DDF
-P 5300 3225
-F 0 "#PWR06" H 5300 3075 50  0001 C CNN
-F 1 "+3.3V" H 5300 3375 50  0000 C CNN
-F 2 "" H 5300 3225 50  0000 C CNN
-F 3 "" H 5300 3225 50  0000 C CNN
-	1    5300 3225
+P 5325 3225
+F 0 "#PWR06" H 5325 3075 50  0001 C CNN
+F 1 "+3.3V" H 5325 3375 50  0000 C CNN
+F 2 "" H 5325 3225 50  0000 C CNN
+F 3 "" H 5325 3225 50  0000 C CNN
+	1    5325 3225
 	1    0    0    -1
 $EndComp
@@
 L device:R R3
 U 1 1 5EEE416B
-P 5225 4775
-F 0 "R3" V 5225 4775 50  0000 C CNN
-F 1 "470" V 5175 4975 50  0000 C CNN
-F 2 "" V 5155 4775 50  0000 C CNN
-F 3 "" H 5225 4775 50  0000 C CNN
-	1    5225 4775
+P 5100 4775
+F 0 "R3" V 5100 4775 50  0000 C CNN
+F 1 "470" V 5050 4975 50  0000 C CNN
+F 2 "" V 5030 4775 50  0000 C CNN
+F 3 "" H 5100 4775 50  0000 C CNN
+	1    5100 4775
 	0    -1   1    0
 $EndComp
@@
 NoConn ~ 5450 4275
 $Comp
-L device:R R1
-U 1 1 5EEE8270
-P 3300 4375
-F 0 "R1" H 3400 4425 50  0000 L CNN
-F 1 "680" H 3400 4325 50  0000 L CNN
-F 2 "" V 3230 4375 50  0000 C CNN
-F 3 "" H 3300 4375 50  0000 C CNN
-	1    3300 4375
-	1    0    0    -1
-$EndComp
-$Comp
 L device:R R6
 U 1 1 5EEE8D51
@@
 L device:R R4
 U 1 1 5EF77CF6
-P 5225 4875
-F 0 "R4" V 5225 4875 50  0000 C CNN
-F 1 "470" V 5175 5075 50  0000 C CNN
-F 2 "" V 5155 4875 50  0000 C CNN
-F 3 "" H 5225 4875 50  0000 C CNN
-	1    5225 4875
+P 5100 4875
+F 0 "R4" V 5100 4875 50  0000 C CNN
+F 1 "470" V 5050 5075 50  0000 C CNN
+F 2 "" V 5030 4875 50  0000 C CNN
+F 3 "" H 5100 4875 50  0000 C CNN
+	1    5100 4875
 	0    -1   1    0
 $EndComp
@@
 L device:R R5
 U 1 1 5EF787E4
-P 5225 4975
-F 0 "R5" V 5225 4975 50  0000 C CNN
-F 1 "470" V 5175 5175 50  0000 C CNN
-F 2 "" V 5155 4975 50  0000 C CNN
-F 3 "" H 5225 4975 50  0000 C CNN
-	1    5225 4975
+P 5100 4975
+F 0 "R5" V 5100 4975 50  0000 C CNN
+F 1 "470" V 5050 5175 50  0000 C CNN
+F 2 "" V 5030 4975 50  0000 C CNN
+F 3 "" H 5100 4975 50  0000 C CNN
+	1    5100 4975
 	0    -1   1    0
 $EndComp
@@
 L device:R R2
 U 1 1 5EF7A4FE
-P 5225 4675
-F 0 "R2" V 5225 4675 50  0000 C CNN
-F 1 "470" V 5275 4475 50  0000 C CNN
-F 2 "" V 5155 4675 50  0000 C CNN
-F 3 "" H 5225 4675 50  0000 C CNN
-	1    5225 4675
+P 5100 4675
+F 0 "R2" V 5100 4675 50  0000 C CNN
+F 1 "470" V 5150 4475 50  0000 C CNN
+F 2 "" V 5030 4675 50  0000 C CNN
+F 3 "" H 5100 4675 50  0000 C CNN
+	1    5100 4675
 	0    1    -1   0
 $EndComp
@@
 Connection ~ 3300 3075
 Wire Wire Line
-	5075 4975 4900 4975
-Wire Wire Line
-	5075 4875 4500 4875
+	4950 4975 4900 4975
+Wire Wire Line
+	4950 4875 4500 4875
 Wire Wire Line
 	4900 5475 4900 5525
@@
 	5650 2275 5650 2425
 Wire Wire Line
-	3100 2025 3100 2075
-Wire Wire Line
-	3100 2075 3100 2225
-Wire Wire Line
-	3300 1825 3300 2075
-Wire Wire Line
-	3300 2075 3300 2225
+	3100 2025 3100 2225
+Wire Wire Line
+	3300 1825 3300 2225
 Wire Wire Line
 	3300 1825 3250 1825
 Wire Wire Line
-	8450 3775 8450 4875
-Wire Wire Line
-	8450 4875 8450 5525
-Wire Wire Line
-	3300 2625 3300 3075
-Wire Wire Line
-	3300 3075 3300 3475
-Wire Wire Line
-	3300 3475 3300 4225
-Connection ~ 3300 3475
+	8450 3775 8450 5525
 Wire Wire Line
 	5950 2425 5950 3775
@@
 	6950 4275 7000 4275
 Wire Wire Line
-	5450 4475 5300 4475
-Wire Wire Line
-	3700 4675 5075 4675
+	5250 4475 5450 4475
+Wire Wire Line
+	3700 4675 4950 4675
 Wire Wire Line
 	3700 5475 3700 5525
@@
 	3300 5475 3300 5525
 Wire Wire Line
-	3300 4525 3300 5075
-Wire Wire Line
-	3200 3475 3300 3475
-Wire Wire Line
-	3300 3475 3950 3475
-Wire Wire Line
-	5300 4475 5300 3225
+	3300 4475 3300 5075
+Wire Wire Line
+	3200 3475 3950 3475
+Wire Wire Line
+	5325 4475 5325 3225
 Wire Wire Line
 	7900 4575 8600 4575
@@
 Connection ~ 8450 4875
 Wire Wire Line
-	7350 5025 7350 5075
-Wire Wire Line
-	7350 5075 7350 5125
+	7350 5025 7350 5125
 Wire Wire Line
 	6950 5075 7350 5075
@@
 ferrite ring
 Wire Wire Line
-	7450 3225 7450 3675
-Wire Wire Line
-	7450 3675 7450 4475
+	7450 3225 7450 4475
 Wire Wire Line
 	7450 4475 6950 4475
@@
 	5560 1905 5420 1905
 Wire Wire Line
-	5375 4675 5450 4675
-Wire Wire Line
-	5375 4875 5450 4875
-Wire Wire Line
-	5450 4975 5375 4975
+	5250 4675 5450 4675
+Wire Wire Line
+	5250 4875 5450 4875
+Wire Wire Line
+	5450 4975 5250 4975
 Wire Wire Line
 	3950 3475 3950 3200
 $Comp
-L pzs_devices:LED-CIRCLE D3
+L pzs_devices:LED-CIRCLE D2
 U 1 1 5EF86B1D
 P 3300 5275
-F 0 "D3" V 3300 5450 50  0000 C CNN
+F 0 "D2" V 3300 5450 50  0000 C CNN
 F 1 "white" V 3450 5350 50  0000 L CNN
 F 2 "" H 3300 5275 50  0000 C CNN
@@
 $EndComp
 $Comp
-L pzs_devices:LED-CIRCLE D4
+L pzs_devices:LED-CIRCLE D3
 U 1 1 5EF8710B
 P 3700 5275
-F 0 "D4" V 3700 5450 50  0000 C CNN
+F 0 "D3" V 3700 5450 50  0000 C CNN
 F 1 "blue" V 3850 5350 50  0000 L CNN
 F 2 "" H 3700 5275 50  0000 C CNN
@@
 $EndComp
 $Comp
-L pzs_devices:LED-CIRCLE D5
+L pzs_devices:LED-CIRCLE D4
 U 1 1 5EF87176
 P 4100 5275
-F 0 "D5" V 4100 5450 50  0000 C CNN
+F 0 "D4" V 4100 5450 50  0000 C CNN
 F 1 "green" V 4250 5350 50  0000 L CNN
 F 2 "" H 4100 5275 50  0000 C CNN
@@
 $EndComp
 $Comp
-L pzs_devices:LED-CIRCLE D6
+L pzs_devices:LED-CIRCLE D5
 U 1 1 5EF871E6
 P 4500 5275
-F 0 "D6" V 4500 5450 50  0000 C CNN
+F 0 "D5" V 4500 5450 50  0000 C CNN
 F 1 "yellow" V 4650 5350 50  0000 L CNN
 F 2 "" H 4500 5275 50  0000 C CNN
@@
 $EndComp
 $Comp
-L pzs_devices:LED-CIRCLE D7
+L pzs_devices:LED-CIRCLE D6
 U 1 1 5EF8725D
 P 4900 5275
-F 0 "D7" V 4900 5450 50  0000 C CNN
+F 0 "D6" V 4900 5450 50  0000 C CNN
 F 1 "red" V 5050 5350 50  0000 L CNN
 F 2 "" H 4900 5275 50  0000 C CNN
@@
 	4900 3525 4900 3275
 Wire Wire Line
-	6950 4675 7625 4675
-Wire Wire Line
-	7625 4675 8600 4675
-Wire Wire Line
-	7900 3225 7900 4075
-Wire Wire Line
-	7900 4075 7900 4575
+	6950 4675 8600 4675
+Wire Wire Line
+	7900 3225 7900 4575
 Wire Wire Line
 	7625 4675 7625 4475
@@
 NoConn ~ 6950 4575
 Wire Wire Line
-	5375 4775 5450 4775
+	5250 4775 5450 4775
 Wire Wire Line
 	4900 4975 4900 5075
@@
 	4100 5075 4100 4775
 Wire Wire Line
-	4100 4775 5075 4775
+	4100 4775 4950 4775
 Wire Wire Line
 	3700 5075 3700 4675
+$Comp
+L device:R R1
+U 1 1 5F021C4E
+P 5100 4475
+F 0 "R1" V 5100 4475 50  0000 C CNN
+F 1 "470" V 5150 4275 50  0000 C CNN
+F 2 "" V 5030 4475 50  0000 C CNN
+F 3 "" H 5100 4475 50  0000 C CNN
+	1    5100 4475
+	0    1    -1   0
+$EndComp
+Connection ~ 5325 4475
+Wire Wire Line
+	4950 4475 3300 4475
+Wire Wire Line
+	3300 2625 3300 3475
+Connection ~ 3300 3475
 $EndSCHEMATC

Commit message: 200714
Parts:
- removed C1: 100n, symbol device:C_Small
- removed D1: 1N4001, symbol pzs_others:diode
- removed L1: EMI_Filter_LL, symbol device:EMI_Filter_LL
- removed P1: BNC, symbol mm7d-rescue:BNC
- removed P2: DB9, symbol mm7d-rescue:DB9
- removed Sp1: Speaker Crystal, symbol device:Speaker_Ultrasound
- removed U1: Adafruit Huzzah Breakout, symbol pzs_devices:Adafruit_Huzzah_Breakout
- added D101: 1N4001, Diodes_THT:Diode_DO-41_SOD81_Horizontal_RM10, symbol D
- added P101, P102: CONN_01X02, Socket_Strips:Socket_Strip_Straight_1x02, symbol CONN_01X02
- added U101-JP4, U101-JP5: CONN_01X10, Socket_Strips:Socket_Strip_Straight_1x10, symbol CONN_01X10
- C101: renamed from C2; value 1000u -> 470u; footprint (none) -> Capacitors_THT:C_Radial_D8_L11.5_P3.5
- C102: renamed from C3; footprint (none) -> Capacitors_THT:C_Rect_L7_W4.5_P5
- D102: renamed from D2; footprint (none) -> LEDs:LED-3MM
- D103: renamed from D3; footprint (none) -> LEDs:LED-3MM
- D104: renamed from D4; footprint (none) -> LEDs:LED-3MM
- D105: renamed from D5; footprint (none) -> LEDs:LED-3MM
- D106: renamed from D6; footprint (none) -> LEDs:LED-3MM
- R101: renamed from R1; footprint (none) -> Resistors_THT:Resistor_Horizontal_RM7mm
- R102: renamed from R2; footprint (none) -> Resistors_THT:Resistor_Horizontal_RM7mm
- R103: renamed from R3; footprint (none) -> Resistors_THT:Resistor_Horizontal_RM7mm
- R104: renamed from R4; footprint (none) -> Resistors_THT:Resistor_Horizontal_RM7mm
- R105: renamed from R5; footprint (none) -> Resistors_THT:Resistor_Horizontal_RM7mm
- R106: renamed from R6; footprint (none) -> Resistors_THT:Resistor_Horizontal_RM7mm
- R107: renamed from R7; footprint (none) -> Resistors_THT:Resistor_Horizontal_RM10mm
- R108: renamed from R8; footprint (none) -> Resistors_THT:Resistor_Horizontal_RM10mm
- U102: renamed from U2; footprint (none) -> Socket_Strips:Socket_Strip_Straight_1x04
- U103: renamed from U3; footprint (none) -> Socket_Strips:Socket_Strip_Straight_1x04
Connections:
- net +3V3: now also R101.2, U101-JP5.3 (P3); no longer R101.1
- net +5V: now also D101.1 (K), P101.2 (P2), U101-JP4.8 (P8)
- net GND: now also D101.2 (A), P101.1 (P1), P102.1 (P1), U101-JP4.10 (P10)
- net at R107.2, R108.1: now also U101-JP4.2 (P2)
- net at C102.1: now also U101-JP4.5 (P5)
- net at R106.2, U103.2 (IO): now also U101-JP4.6 (P6)
- net at R102.1: now also D103.2 (A)
- net at R103.2: now also D104.2 (A)
- net at R104.2: now also D105.2 (A)
- net at R105.2: now also D106.2 (A)
- net at R103.1: now also U101-JP5.6 (P6); no longer D104.2 (A)
- net at R104.1: now also U101-JP5.7 (P7); no longer D105.2 (A)
- net at R105.1: now also U101-JP5.8 (P8); no longer D106.2 (A)
- net at R102.2: now also U101-JP5.5 (P5); no longer D103.2 (A)
- net at D102.2 (A): now also R101.1; no longer R101.2
- net at C102.2: now also P102.2 (P2)
- no-connect marks 21 -> 11
Other:
- note added: "5V DC"
- note added: "Adafruit\nHuzzah\nBreakout"
- note added: "Piezo speaker"
- note added: "U101"
- note removed: "5V DC in"
- note removed: "Console (3,3V serial)"
- note removed: "PCB"
- note removed: "ferrite ring"
- moved on the sheet: C101, C102, D102, D103, D104, D105, D106, R101, R102, R103, R104, R105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
