File: cad_files/mm7d/mm7d.sch (KiCad schematic (older format))
At the start: 22 parts, among them P101 CONN_01X02, P102 CONN_01X02, U101-JP4 CONN_01X10, U101-JP5 CONN_01X10, U102 MQ-135M, U103 DHT11

Commit message: 230317
Parts:
- removed U102: MQ-135M, Socket_Strips:Socket_Strip_Straight_1x04, symbol pzs_devices:MQ-135M
- C101, C102: symbol device:CP_Small -> mm7d-rescue:device_CP_Small
- D101: symbol D -> mm7d-rescue:D
- D102, D103, D104, D105, D106: symbol pzs_devices:LED-CIRCLE -> mm7d-rescue:pzs_devices_LED-CIRCLE
- P101, P102: symbol CONN_01X02 -> mm7d-rescue:CONN_01X02
- R101, R102, R103, R104, R105, R106: symbol device:R -> mm7d-rescue:device_R
- R107: value 39k -> 5.1k; symbol device:R -> mm7d-rescue:device_R
- R108: value 9.1k -> 750; symbol device:R -> mm7d-rescue:device_R
- U101-JP4, U101-JP5: symbol CONN_01X10 -> mm7d-rescue:CONN_01X10
- U102: renamed from U103; symbol pzs_devices:DHT11 -> mm7d-rescue:pzs_devices_DHT11
Connections:
- net +5V: now also R107.1
- no-connect marks 11 -> 10
Other:
- moved on the sheet: C101, C102, D101, D102, D103, D104, D105, D106, P101, P102, R101, R102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
