File: cad_files/wiring/wiring.sch (KiCad schematic (older format))
At the start: 7 parts, among them P1 SN10M 5.5/2.1, P101 CONN_01X02, P102 CONN_01X02, P2 DB9F, U101-JP1 CONN_01X06

Commit message: 200716
Other:
- note added: "+"
Changed lines of the file:
@@
 LIBS:contrib
 LIBS:valves
-LIBS:connectors-cache
+LIBS:wiring-cache
 EELAYER 25 0
 EELAYER END
@@
 Rev "200620"
 Comp "Pozsar Zsolt - http://www.szerafingomba.hu"
-Comment1 "Connectors"
+Comment1 "Internal wiring"
 Comment2 ""
 Comment3 ""
@@
 Text Notes 6450 2800 0    60   ~ 0
 Console
+Text Notes 4700 3100 0    60   ~ 0
++
 $EndSCHEMATC
