File: cad_files/wiring/wiring.sch (KiCad schematic (older format))
At the start: 7 parts, among them P1 SN10M 5.5/2.1, P101 CONN_01X02, P102 CONN_01X02, P2 DB9F, U101-JP1 CONN_01X06

Commit message: 230317
Parts:
- C1: symbol C -> wiring-rescue:C
- LS1: symbol Speaker_Crystal -> wiring-rescue:Speaker_Crystal
- P1: symbol BNC -> wiring-rescue:BNC
- P101, P102: symbol CONN_01X02 -> wiring-rescue:CONN_01X02
- P2: symbol DB9 -> wiring-rescue:DB9
- U101-JP1: symbol CONN_01X06 -> wiring-rescue:CONN_01X06
Changed lines of the file:
@@
-EESchema Schematic File Version 2
-LIBS:power
-LIBS:device
-LIBS:transistors
-LIBS:conn
-LIBS:linear
-LIBS:regul
-LIBS:74xx
-LIBS:cmos4000
-LIBS:adc-dac
-LIBS:memory
-LIBS:xilinx
-LIBS:microcontrollers
-LIBS:dsp
-LIBS:microchip
-LIBS:analog_switches
-LIBS:motorola
-LIBS:texas
-LIBS:intel
-LIBS:audio
-LIBS:interface
-LIBS:digital-audio
-LIBS:philips
-LIBS:display
-LIBS:cypress
-LIBS:siliconi
-LIBS:opto
-LIBS:atmel
-LIBS:contrib
-LIBS:valves
-LIBS:wiring-cache
-EELAYER 25 0
+EESchema Schematic File Version 4
+EELAYER 30 0
 EELAYER END
 $Descr A4 11693 8268
 encoding utf-8
 Sheet 1 1
-Title "MM7D Air quality measuring device"
-Date "2020-06-20"
-Rev "200620"
-Comp "Pozsar Zsolt - http://www.szerafingomba.hu"
+Title "MM7D RH/T measuring device"
+Date "2024-03-17"
+Rev "231006"
+Comp "Pozsar Zsolt - http://www.pozsarzs.hu"
 Comment1 "Internal wiring"
 Comment2 ""
 Comment3 ""
-Comment4 "Draw no.: 59/12/6"
+Comment4 ""
 $EndDescr
 $Comp
-L BNC P1
+L wiring-rescue:BNC P1
 U 1 1 5F0F33AE
 P 4550 3100
@@
 $EndComp
 $Comp
-L C C1
+L wiring-rescue:C C1
 U 1 1 5F0F33F6
 P 4750 3550
@@
 $EndComp
 $Comp
-L CONN_01X02 P101
+L wiring-rescue:CONN_01X02 P101
 U 1 1 5F0F3457
 P 4600 4450
@@
 $EndComp
 $Comp
-L CONN_01X02 P102
+L wiring-rescue:CONN_01X02 P102
 U 1 1 5F0F3486
 P 5600 4450
@@
 $EndComp
 $Comp
-L DB9 P2
+L wiring-rescue:DB9 P2
 U 1 1 5F0F34AD
 P 6650 3100
@@
 $EndComp
 $Comp
-L CONN_01X06 U101-JP1
+L wiring-rescue:CONN_01X06 U101-JP1
 U 1 1 5F0F34CC
 P 6800 4450
@@
 $EndComp
 $Comp
-L Speaker_Crystal LS1
+L wiring-rescue:Speaker_Crystal LS1
 U 1 1 5F0F34FF
 P 5550 3750
@@
 $EndComp
 Wire Wire Line
-	4550 3300 4550 4250
+	4550 3300 4550 3550
 Wire Wire Line
 	4600 3550 4550 3550
@@
 	4950 4200 4650 4200
 Wire Wire Line
-	4950 3100 4950 4200
+	4950 3100 4950 3550
 Wire Wire Line
 	4950 3550 4900 3550
@@
 Text Notes 4700 3100 0    60   ~ 0
 +
+Wire Wire Line
+	4550 3550 4550 4250
+Wire Wire Line
+	4950 3550 4950 4200
 $EndSCHEMATC
